File: tests/sample_project/sample.kicad_pcb (KiCad board)
At the start: 2 copper layers, 30 x 20 mm, 2 parts

Commit message: fix: edited sample projects
Parts:
- C1: footprint Capacitor_SMD:C_0603_1608Metric -> C_0603_1608Metric
- R1: footprint Resistor_SMD:R_0603_1608Metric -> R_0603_1608Metric
